File: audio sense board rv1.sch (EAGLE design)
At the start: 32 parts, among them IC2 TSOP38238, J1 PJRAN1X1U01X, J4 PJRAN1X1U01X, Q1 2N3904, Q2 2N3904

Commit message: rework led and signals
Parts:
- removed DEBUG: Debug Jumper, SparkFun-Connectors:CONN_02LOCK
- removed R7: 10K, Samac Populated:CRCW120610K0FKEAC
Connections:
- removed net N$12: ARDUINOMICRO.A2, D2.A, Q2.C, R8.1
- removed net N$2: ARDUINOMICRO.A1, D1.A, Q1.C, R1.1
- new net J1SIGNAL: ARDUINOMICRO.A1, D1.A, R1.1
- new net J4SIGNAL: ARDUINOMICRO.A2, D2.A, R8.1
- new net N$8: D1.C, Q1.C
- net GND: no longer DEBUG.2
- net N$5: now also Q2.C; no longer ARDUINOMICRO.A0, D1.C, DEBUG.1, R7.1
- net VCC: no longer R7.2
Other:
- moved on the sheet: D1, D2, R1, R10, R12, R3, R5, R8
